File: pcb/m5-pantilt-v1.0/m5-pantilt.kicad_pcb (KiCad board)
At the start: 2 copper layers, 50 x 50 mm, 39 parts, among them J1 Conn_02x15_Odd_Even, J2 Conn_02x15_Odd_Even, J3 Conn_01x03, J5 BAT, J6 Conn_01x04, J7 5V_POWER, J8 Conn_01x03, Q1 IRLML6402, Q2 BC857, SW1 SW_SPDT, U1 MAX3485

Commit message: PCB manufacture fixes: (1) assign LCSC parts C160259 (J3/J8 JST EH 3P) and C157926 (J6 JST PH 4P side, both verified via JLC API), mark J1/J2/SW1 as consigned with purchase specs; (2) exclude Hole1-4 mounting holes, R9-R12 PWM jumpers and consigned parts from CPL; (3) fix assembly types J1=SMD-footprint, J3/J5/J6/J8/J7=THT in BOM CSV; (4) fix U1 footprint wide SO-8 -> narrow SOIC-8_3.9x4.9mm (C668204 is narrow-body SOP-8), move 9 track endpoints, DRC connectivity clean, regenerate gerbers/CPL/zip; update BOM.md, manufacture README and route doc
Parts:
- U1: footprint Package_SO:SO-8_5.3x6.2mm_P1.27mm -> Package_SO:SOIC-8_3.9x4.9mm_P1.27mm
Routing:
- net /TXD2: track 17.6 -> 18.6 mm
- net /RXD2: track 23.4 -> 24.4 mm
- net /TTL: track 6.39 -> 7.42 mm
- net GND: track 2.50 -> 3.52 mm
- net +3V3: track 39.7 -> 40.8 mm
- net Net-(U1-B): track 6.40 -> 7.40 mm
- net Net-(Q2-C): track 6.88 -> 7.86 mm
