File: pcb/m5-pantilt-v1.0/m5-pantilt.kicad_pcb (KiCad board)
At the start: 2 copper layers, 50 x 50 mm, 39 parts, among them J1 Conn_02x15_Odd_Even, J2 Conn_02x15_Odd_Even, J3 Conn_01x03, J5 BAT, J6 Conn_01x04, J7 5V_POWER, J8 Conn_01x03, Q1 IRLML6402, Q2 BC857, SW1 SW_SPDT, U1 MAX3485

Commit message: Eliminate all DRC/parity warnings: move 34 board footprints into project library m5-pantilt.pretty (pads/tracks/nets untouched; Q1 custom SOT-23 pads -> SOT-23_HandSolder_Pads, mirrored R1/R2/R5 variants get _Mirrored suffix, FPIDs + schematic Footprint fields repointed), clip J6/SW1 out-of-board silkscreen to 0.4mm inside edges, shorten 2 J1 back ticks crossing decorative frame; rebuild manufacture outputs via KiCad 10.0.7 pipeline. Result: DRC 0 errors/0 warnings/0 unconnected, schematic parity 0 warnings, ERC 0 errors/59 warnings (official legacy symbol metadata only, footprint_link 33->1). Update checks/README.md resolution table and manufacture docs
Parts:
- C1, C2, C3, C4: footprint Capacitor_SMD:C_1206_3216Metric_Pad1.33x1.80mm_HandSolder -> m5-pantilt:C_1206_3216Metric_Pad1.33x1.80mm_HandSolder
- C5: footprint Capacitor_SMD:C_0603_1608Metric -> m5-pantilt:C_0603_1608Metric
- D1: footprint Diode_SMD:D_SMA -> m5-pantilt:D_SMA
- D2: footprint Diode_SMD:D_SOD-128 -> m5-pantilt:D_SOD-128
- J1: footprint Connector_PinHeader_2.54mm:PinHeader_2x15_P2.54mm_Vertical_SMD -> m5-pantilt:PinHeader_2x15_P2.54mm_Vertical_SMD
- J2: footprint Connector_PinSocket_2.54mm:PinSocket_2x15_P2.54mm_Vertical_SMD -> m5-pantilt:PinSocket_2x15_P2.54mm_Vertical_SMD
- J3, J8: footprint Connector_JST:JST_EH_B3B-EH-A_1x03_P2.50mm_Vertical -> m5-pantilt:JST_EH_B3B-EH-A_1x03_P2.50mm_Vertical
- J5: footprint Connector_JST:JST_PH_B2B-PH-K_1x02_P2.00mm_Vertical -> m5-pantilt:JST_PH_B2B-PH-K_1x02_P2.00mm_Vertical
- J6: footprint Connector_JST:JST_PH_S4B-PH-K_1x04_P2.00mm_Horizontal -> m5-pantilt:JST_PH_S4B-PH-K_1x04_P2.00mm_Horizontal
- J7: footprint Connector_JST:JST_XH_B2B-XH-A_1x02_P2.50mm_Vertical -> m5-pantilt:JST_XH_B2B-XH-A_1x02_P2.50mm_Vertical
- Q1: footprint Package_TO_SOT_SMD:SOT-23 -> m5-pantilt:SOT-23_HandSolder_Pads
- Q2: footprint Package_TO_SOT_SMD:SOT-23 -> m5-pantilt:SOT-23
- R1, R2: footprint Resistor_SMD:R_0603_1608Metric -> m5-pantilt:R_0603_1608Metric_Mirrored
- R10, R11, R12, R3, R4, R9: footprint Resistor_SMD:R_0603_1608Metric_Pad0.98x0.95mm_HandSolder -> m5-pantilt:R_0603_1608Metric_Pad0.98x0.95mm_HandSolder
- R13, R14, R15, R6, R7, R8: footprint Resistor_SMD:R_0603_1608Metric -> m5-pantilt:R_0603_1608Metric
- R5: footprint Resistor_SMD:R_0603_1608Metric_Pad0.98x0.95mm_HandSolder -> m5-pantilt:R_0603_1608Metric_Pad0.98x0.95mm_HandSolder_Mirrored
- REF**: footprint Symbol:OSHW-Logo2_7.3x6mm_SilkScreen -> m5-pantilt:OSHW-Logo2_7.3x6mm_SilkScreen
- SW1: footprint Button_Switch_THT:SW_CuK_OS102011MA1QN1_SPDT_Angled -> m5-pantilt:SW_CuK_OS102011MA1QN1_SPDT_Angled
- U1: footprint Package_SO:SOIC-8_3.9x4.9mm_P1.27mm -> m5-pantilt:SOIC-8_3.9x4.9mm_P1.27mm
