File: pcb/m5-pantilt-v1.0/m5-pantilt.kicad_sch (KiCad schematic)
At the start: 33 parts, among them J1 Conn_02x15_Odd_Even, J2 Conn_02x15_Odd_Even, J3 Conn_01x03, J5 BAT, J6 Conn_01x04, J7 5V_POWER, J8 Conn_01x03, Q1 IRLML6402, Q2 BC857, SW1 SW_SPDT, U1 MAX3485

Commit message: PCB manufacture fixes: (1) assign LCSC parts C160259 (J3/J8 JST EH 3P) and C157926 (J6 JST PH 4P side, both verified via JLC API), mark J1/J2/SW1 as consigned with purchase specs; (2) exclude Hole1-4 mounting holes, R9-R12 PWM jumpers and consigned parts from CPL; (3) fix assembly types J1=SMD-footprint, J3/J5/J6/J8/J7=THT in BOM CSV; (4) fix U1 footprint wide SO-8 -> narrow SOIC-8_3.9x4.9mm (C668204 is narrow-body SOP-8), move 9 track endpoints, DRC connectivity clean, regenerate gerbers/CPL/zip; update BOM.md, manufacture README and route doc
Parts:
- U1: footprint Package_SO:SO-8_5.3x6.2mm_P1.27mm -> Package_SO:SOIC-8_3.9x4.9mm_P1.27mm
Changed lines of the file:
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@@
       (effects (font (size 1.27 1.27)))
     )
-    (property "Footprint" "Package_SO:SO-8_5.3x6.2mm_P1.27mm" (at 123.19 153.67 0)
+    (property "Footprint" "Package_SO:SOIC-8_3.9x4.9mm_P1.27mm" (at 123.19 153.67 0)
       (effects (font (size 1.27 1.27)) hide)
     )

Commit message: Eliminate all DRC/parity warnings: move 34 board footprints into project library m5-pantilt.pretty (pads/tracks/nets untouched; Q1 custom SOT-23 pads -> SOT-23_HandSolder_Pads, mirrored R1/R2/R5 variants get _Mirrored suffix, FPIDs + schematic Footprint fields repointed), clip J6/SW1 out-of-board silkscreen to 0.4mm inside edges, shorten 2 J1 back ticks crossing decorative frame; rebuild manufacture outputs via KiCad 10.0.7 pipeline. Result: DRC 0 errors/0 warnings/0 unconnected, schematic parity 0 warnings, ERC 0 errors/59 warnings (official legacy symbol metadata only, footprint_link 33->1). Update checks/README.md resolution table and manufacture docs
Parts:
- C1, C2, C3, C4: footprint Capacitor_SMD:C_1206_3216Metric_Pad1.33x1.80mm_HandSolder -> m5-pantilt:C_1206_3216Metric_Pad1.33x1.80mm_HandSolder
- C5: footprint Capacitor_SMD:C_0603_1608Metric -> m5-pantilt:C_0603_1608Metric
- D1: footprint Diode_SMD:D_SMA -> m5-pantilt:D_SMA
- D2: footprint Diode_SMD:D_SOD-128 -> m5-pantilt:D_SOD-128
- J1: footprint Connector_PinHeader_2.54mm:PinHeader_2x15_P2.54mm_Vertical_SMD -> m5-pantilt:PinHeader_2x15_P2.54mm_Vertical_SMD
- J2: footprint Connector_PinSocket_2.54mm:PinSocket_2x15_P2.54mm_Vertical_SMD -> m5-pantilt:PinSocket_2x15_P2.54mm_Vertical_SMD
- J3, J8: footprint Connector_JST:JST_EH_B3B-EH-A_1x03_P2.50mm_Vertical -> m5-pantilt:JST_EH_B3B-EH-A_1x03_P2.50mm_Vertical
- J5: footprint Connector_JST:JST_PH_B2B-PH-K_1x02_P2.00mm_Vertical -> m5-pantilt:JST_PH_B2B-PH-K_1x02_P2.00mm_Vertical
- J6: footprint Connector_JST:JST_PH_S4B-PH-K_1x04_P2.00mm_Horizontal -> m5-pantilt:JST_PH_S4B-PH-K_1x04_P2.00mm_Horizontal
- J7: footprint Connector_JST:JST_XH_B2B-XH-A_1x02_P2.50mm_Vertical -> m5-pantilt:JST_XH_B2B-XH-A_1x02_P2.50mm_Vertical
- Q1: footprint Package_TO_SOT_SMD:SOT-23 -> m5-pantilt:SOT-23
- Q2: footprint Package_TO_SOT_SMD:SOT-23 -> m5-pantilt:SOT-23_Mirrored
- R1, R2: footprint Resistor_SMD:R_0603_1608Metric -> m5-pantilt:R_0603_1608Metric_Mirrored
- R10, R11, R12, R3, R4, R9: footprint Resistor_SMD:R_0603_1608Metric_Pad0.98x0.95mm_HandSolder -> m5-pantilt:R_0603_1608Metric_Pad0.98x0.95mm_HandSolder
- R13, R14, R15, R6, R7, R8: footprint Resistor_SMD:R_0603_1608Metric -> m5-pantilt:R_0603_1608Metric
- R5: footprint Resistor_SMD:R_0603_1608Metric_Pad0.98x0.95mm_HandSolder -> m5-pantilt:R_0603_1608Metric_Pad0.98x0.95mm_HandSolder_Mirrored
- SW1: footprint Button_Switch_THT:SW_CuK_OS102011MA1QN1_SPDT_Angled -> m5-pantilt:SW_CuK_OS102011MA1QN1_SPDT_Angled
- U1: footprint Package_SO:SOIC-8_3.9x4.9mm_P1.27mm -> m5-pantilt:SOIC-8_3.9x4.9mm_P1.27mm
Changed lines of the file:
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@@
       (effects (font (size 1.27 1.27)))
     )
-    (property "Footprint" "Connector_PinHeader_2.54mm:PinHeader_2x15_P2.54mm_Vertical_SMD" (at 90.17 86.36 0)
+    (property "Footprint" "m5-pantilt:PinHeader_2x15_P2.54mm_Vertical_SMD" (at 90.17 86.36 0)
       (effects (font (size 1.27 1.27)) hide)
     )
@@
       (effects (font (size 1.27 1.27)))
     )
-    (property "Footprint" "Connector_JST:JST_PH_B2B-PH-K_1x02_P2.00mm_Vertical" (at 20.32 138.43 0)
+    (property "Footprint" "m5-pantilt:JST_PH_B2B-PH-K_1x02_P2.00mm_Vertical" (at 20.32 138.43 0)
       (effects (font (size 1.27 1.27)) hide)
     )
@@
       (effects (font (size 1.27 1.27)) (justify left))
     )
-    (property "Footprint" "Resistor_SMD:R_0603_1608Metric_Pad0.98x0.95mm_HandSolder" (at 205.74 97.282 90)
+    (property "Footprint" "m5-pantilt:R_0603_1608Metric_Pad0.98x0.95mm_HandSolder" (at 205.74 97.282 90)
       (effects (font (size 1.27 1.27)) hide)
     )
@@
       (effects (font (size 1.27 1.27)) (justify left))
     )
-    (property "Footprint" "Resistor_SMD:R_0603_1608Metric_Pad0.98x0.95mm_HandSolder" (at 205.74 123.952 90)
+    (property "Footprint" "m5-pantilt:R_0603_1608Metric_Pad0.98x0.95mm_HandSolder" (at 205.74 123.952 90)
       (effects (font (size 1.27 1.27)) hide)
     )
@@
       (effects (font (size 1.27 1.27)) (justify left))
     )
-    (property "Footprint" "Connector_JST:JST_PH_S4B-PH-K_1x04_P2.00mm_Horizontal" (at 149.86 81.28 0)
+    (property "Footprint" "m5-pantilt:JST_PH_S4B-PH-K_1x04_P2.00mm_Horizontal" (at 149.86 81.28 0)
       (effects (font (size 1.27 1.27)) hide)
     )
@@
       (effects (font (size 1.27 1.27)))
     )
-    (property "Footprint" "Capacitor_SMD:C_1206_3216Metric_Pad1.33x1.80mm_HandSolder" (at 218.7448 83.82 0)
+    (property "Footprint" "m5-pantilt:C_1206_3216Metric_Pad1.33x1.80mm_HandSolder" (at 218.7448 83.82 0)
       (effects (font (size 1.27 1.27)) hide)
     )
@@
       (effects (font (size 1.27 1.27)))
     )
-    (property "Footprint" "Button_Switch_THT:SW_CuK_OS102011MA1QN1_SPDT_Angled" (at 34.29 156.21 0)
+    (property "Footprint" "m5-pantilt:SW_CuK_OS102011MA1QN1_SPDT_Angled" (at 34.29 156.21 0)
       (effects (font (size 1.27 1.27)) hide)
     )
@@
       (effects (font (size 1.27 1.27)))
     )
-    (property "Footprint" "Connector_JST:JST_XH_B2B-XH-A_1x02_P2.50mm_Vertical" (at 20.32 109.22 0)
+    (property "Footprint" "m5-pantilt:JST_XH_B2B-XH-A_1x02_P2.50mm_Vertical" (at 20.32 109.22 0)
       (effects (font (size 1.27 1.27)) hide)
     )
@@
       (effects (font (size 1.27 1.27)))
     )
-    (property "Footprint" "Capacitor_SMD:C_1206_3216Metric_Pad1.33x1.80mm_HandSolder" (at 218.7448 109.22 0)
+    (property "Footprint" "m5-pantilt:C_1206_3216Metric_Pad1.33x1.80mm_HandSolder" (at 218.7448 109.22 0)
       (effects (font (size 1.27 1.27)) hide)
     )
@@
       (effects (font (size 1.27 1.27)))
     )
-    (property "Footprint" "Package_TO_SOT_SMD:SOT-23" (at 42.545 140.97 0)
+    (property "Footprint" "m5-pantilt:SOT-23" (at 42.545 140.97 0)
       (effects (font (size 1.27 1.27) italic) (justify left) hide)
     )
@@
       (effects (font (size 1.27 1.27)) (justify right))
     )
-    (property "Footprint" "Resistor_SMD:R_0603_1608Metric_Pad0.98x0.95mm_HandSolder" (at 36.068 143.51 90)
+    (property "Footprint" "m5-pantilt:R_0603_1608Metric_Pad0.98x0.95mm_HandSolder_Mirrored" (at 36.068 143.51 90)
       (effects (font (size 1.27 1.27)) hide)
     )
@@
       (effects (font (size 1.27 1.27)))
     )
-    (property "Footprint" "Capacitor_SMD:C_1206_3216Metric_Pad1.33x1.80mm_HandSolder" (at 207.3148 83.82 0)
+    (property "Footprint" "m5-pantilt:C_1206_3216Metric_Pad1.33x1.80mm_HandSolder" (at 207.3148 83.82 0)
       (effects (font (size 1.27 1.27)) hide)
     )
@@
       (effects (font (size 1.27 1.27)))
     )
-    (property "Footprint" "Capacitor_SMD:C_1206_3216Metric_Pad1.33x1.80mm_HandSolder" (at 209.2452 116.84 0)
+    (property "Footprint" "m5-pantilt:C_1206_3216Metric_Pad1.33x1.80mm_HandSolder" (at 209.2452 116.84 0)
       (effects (font (size 1.27 1.27)) hide)
     )
@@
       (effects (font (size 1.27 1.27)))
     )
-    (property "Footprint" "Resistor_SMD:R_0603_1608Metric_Pad0.98x0.95mm_HandSolder" (at 220.98 36.322 90)
+    (property "Footprint" "m5-pantilt:R_0603_1608Metric_Pad0.98x0.95mm_HandSolder" (at 220.98 36.322 90)
       (effects (font (size 1.27 1.27)) hide)
     )
@@
       (effects (font (size 1.27 1.27)))
     )
-    (property "Footprint" "Resistor_SMD:R_0603_1608Metric_Pad0.98x0.95mm_HandSolder" (at 220.98 45.212 90)
+    (property "Footprint" "m5-pantilt:R_0603_1608Metric_Pad0.98x0.95mm_HandSolder" (at 220.98 45.212 90)
       (effects (font (size 1.27 1.27)) hide)
     )
@@
       (effects (font (size 1.27 1.27)))
     )
-    (property "Footprint" "Resistor_SMD:R_0603_1608Metric_Pad0.98x0.95mm_HandSolder" (at 220.98 54.102 90)
+    (property "Footprint" "m5-pantilt:R_0603_1608Metric_Pad0.98x0.95mm_HandSolder" (at 220.98 54.102 90)
       (effects (font (size 1.27 1.27)) hide)
     )
@@
       (effects (font (size 1.27 1.27)))
     )
-    (property "Footprint" "Resistor_SMD:R_0603_1608Metric_Pad0.98x0.95mm_HandSolder" (at 220.98 62.992 90)
+    (property "Footprint" "m5-pantilt:R_0603_1608Metric_Pad0.98x0.95mm_HandSolder" (at 220.98 62.992 90)
       (effects (font (size 1.27 1.27)) hide)
     )
@@
       (effects (font (size 1.27 1.27)))
     )
-    (property "Footprint" "Resistor_SMD:R_0603_1608Metric" (at 229.87 97.282 90)
+    (property "Footprint" "m5-pantilt:R_0603_1608Metric" (at 229.87 97.282 90)
       (effects (font (size 1.27 1.27)) hide)
     )
@@
       (effects (font (size 1.27 1.27)))
     )
-    (property "Footprint" "Resistor_SMD:R_0603_1608Metric" (at 229.87 123.952 90)
+    (property "Footprint" "m5-pantilt:R_0603_1608Metric" (at 229.87 123.952 90)
       (effects (font (size 1.27 1.27)) hide)
     )
@@
       (effects (font (size 1.27 1.27)))
     )
-    (property "Footprint" "Package_SO:SOIC-8_3.9x4.9mm_P1.27mm" (at 123.19 153.67 0)
+    (property "Footprint" "m5-pantilt:SOIC-8_3.9x4.9mm_P1.27mm" (at 123.19 153.67 0)
       (effects (font (size 1.27 1.27)) hide)
     )
@@
       (effects (font (size 1.27 1.27)) (justify left))
     )
-    (property "Footprint" "Capacitor_SMD:C_0603_1608Metric" (at 147.0152 130.81 0)
+    (property "Footprint" "m5-pantilt:C_0603_1608Metric" (at 147.0152 130.81 0)
       (effects (font (size 1.27 1.27)) hide)
     )
@@
       (effects (font (size 1.27 1.27)) (justify left))
     )
-    (property "Footprint" "Resistor_SMD:R_0603_1608Metric" (at 155.702 128.27 90)
+    (property "Footprint" "m5-pantilt:R_0603_1608Metric" (at 155.702 128.27 90)
       (effects (font (size 1.27 1.27)) hide)
     )
@@
       (effects (font (size 1.27 1.27)) (justify left))
     )
-    (property "Footprint" "Resistor_SMD:R_0603_1608Metric" (at 155.702 142.24 90)
+    (property "Footprint" "m5-pantilt:R_0603_1608Metric" (at 155.702 142.24 90)
       (effects (font (size 1.27 1.27)) hide)
     )
@@
       (effects (font (size 1.27 1.27)) (justify left))
     )
-    (property "Footprint" "Resistor_SMD:R_0603_1608Metric" (at 93.472 146.05 90)
+    (property "Footprint" "m5-pantilt:R_0603_1608Metric" (at 93.472 146.05 90)
       (effects (font (size 1.27 1.27)) hide)
     )
@@
       (effects (font (size 1.27 1.27)))
     )
-    (property "Footprint" "Diode_SMD:D_SMA" (at 43.18 109.22 0)
+    (property "Footprint" "m5-pantilt:D_SMA" (at 43.18 109.22 0)
       (effects (font (size 1.27 1.27)) hide)
     )
@@
       (effects (font (size 1.27 1.27)))
     )
-    (property "Footprint" "Connector_PinSocket_2.54mm:PinSocket_2x15_P2.54mm_Vertical_SMD" (at 36.83 45.72 0)
+    (property "Footprint" "m5-pantilt:PinSocket_2x15_P2.54mm_Vertical_SMD" (at 36.83 45.72 0)
       (effects (font (size 1.27 1.27)) hide)
     )
@@
       (effects (font (size 1.27 1.27)) (justify left))
     )
-    (property "Footprint" "Connector_JST:JST_EH_B3B-EH-A_1x03_P2.50mm_Vertical" (at 248.92 109.22 0)
+    (property "Footprint" "m5-pantilt:JST_EH_B3B-EH-A_1x03_P2.50mm_Vertical" (at 248.92 109.22 0)
       (effects (font (size 1.27 1.27)) hide)
     )
@@
       (effects (font (size 1.27 1.27)) (justify left))
     )
-    (property "Footprint" "Connector_JST:JST_EH_B3B-EH-A_1x03_P2.50mm_Vertical" (at 248.92 83.82 0)
+    (property "Footprint" "m5-pantilt:JST_EH_B3B-EH-A_1x03_P2.50mm_Vertical" (at 248.92 83.82 0)
       (effects (font (size 1.27 1.27)) hide)
     )
@@
       (effects (font (size 1.27 1.27)) (justify left))
     )
-    (property "Footprint" "Resistor_SMD:R_0603_1608Metric" (at 69.342 120.65 90)
+    (property "Footprint" "m5-pantilt:R_0603_1608Metric_Mirrored" (at 69.342 120.65 90)
       (effects (font (size 1.27 1.27)) hide)
     )
@@
       (effects (font (size 1.27 1.27)))
     )
-    (property "Footprint" "Resistor_SMD:R_0603_1608Metric" (at 81.28 131.318 90)
+    (property "Footprint" "m5-pantilt:R_0603_1608Metric_Mirrored" (at 81.28 131.318 90)
       (effects (font (size 1.27 1.27)) hide)
     )
@@
       (effects (font (size 1.27 1.27)) (justify left))
     )
-    (property "Footprint" "Resistor_SMD:R_0603_1608Metric" (at 135.382 127 90)
+    (property "Footprint" "m5-pantilt:R_0603_1608Metric" (at 135.382 127 90)
       (effects (font (size 1.27 1.27)) hide)
     )
@@
       (effects (font (size 1.27 1.27)) (justify right))
     )
-    (property "Footprint" "Diode_SMD:D_SOD-128" (at 185.42 74.93 0)
+    (property "Footprint" "m5-pantilt:D_SOD-128" (at 185.42 74.93 0)
       (effects (font (size 1.27 1.27)) hide)
     )
@@
       (effects (font (size 1.27 1.27)) (justify left))
     )
-    (property "Footprint" "Package_TO_SOT_SMD:SOT-23" (at 97.79 127.635 0)
+    (property "Footprint" "m5-pantilt:SOT-23_Mirrored" (at 97.79 127.635 0)
       (effects (font (size 1.27 1.27) italic) (justify left) hide)
     )

Commit message: Fix Q1/Q2 schematic Footprint fields (were swapped: Q1 pointed to SOT-23 instead of SOT-23_HandSolder_Pads, Q2 to nonexistent SOT-23_Mirrored) and install KiCad 10 standard symbol library table for the AppImage check environment; rebuild reports. Result: DRC 0/0/0, ERC 59->29 warnings (58 environmental library-table warnings + 1 Q2 missing-footprint warning eliminated; remaining 29 are genuine legacy official symbol versions), schematic parity 41->39 (2 footprint mismatches fixed; remaining 33 field-metadata + 6 mechanical). Correct manufacture/checks docs to the real numbers, including an errata note about the earlier misreported 0-warning parity claim. check-manufacture.py all pass.
Parts:
- Q1: footprint m5-pantilt:SOT-23 -> m5-pantilt:SOT-23_HandSolder_Pads
- Q2: footprint m5-pantilt:SOT-23_Mirrored -> m5-pantilt:SOT-23
Changed lines of the file:
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@@
       (effects (font (size 1.27 1.27)))
     )
-    (property "Footprint" "m5-pantilt:SOT-23" (at 42.545 140.97 0)
+    (property "Footprint" "m5-pantilt:SOT-23_HandSolder_Pads" (at 42.545 140.97 0)
       (effects (font (size 1.27 1.27) italic) (justify left) hide)
     )
@@
       (effects (font (size 1.27 1.27)) (justify left))
     )
-    (property "Footprint" "m5-pantilt:SOT-23_Mirrored" (at 97.79 127.635 0)
+    (property "Footprint" "m5-pantilt:SOT-23" (at 97.79 127.635 0)
       (effects (font (size 1.27 1.27) italic) (justify left) hide)
     )
